Commit message: frames pdf created

File: src/description/roar_bot_description.urdf (robot description, URDF)
Before this commit: robot roar_bot, 4 links, 3 joints
Links:
- added link sensors_link
Joints:
- added joint sensors_joint: type fixed, parent iphone_link, child sensors_link, origin xyz=0.0 0.0 0.0 rpy=3.14 0 0
